File: modules/done-filter/MDL-filter_v2/src/MDL-filter_v2.sch (KiCad schematic (older format))
At the start: 9 parts

Commit message: update modules
Connections:
- net +5V renamed ITF-B_5v
- net GND renamed ITF-A_gnd
- net Output renamed ITF-D_amplified_filtered_signal
Changed lines of the file:
@@
 LIBS:valves
 LIBS:echopen
+LIBS:MDL-filter_v2-cache
 EELAYER 25 0
 EELAYER END
@@
 	1    0    0    -1
 $EndComp
-$Comp
-L +5V #PWR01
-U 1 1 57A4C0CC
-P 2500 3350
-F 0 "#PWR01" H 2500 3200 50  0001 C CNN
-F 1 "+5V" H 2500 3490 50  0000 C CNN
-F 2 "" H 2500 3350 50  0000 C CNN
-F 3 "" H 2500 3350 50  0000 C CNN
-	1    2500 3350
-	1    0    0    -1
-$EndComp
-$Comp
-L GND #PWR02
-U 1 1 57A4C0F0
-P 2500 4100
-F 0 "#PWR02" H 2500 3850 50  0001 C CNN
-F 1 "GND" H 2500 3950 50  0000 C CNN
-F 2 "" H 2500 4100 50  0000 C CNN
-F 3 "" H 2500 4100 50  0000 C CNN
-	1    2500 4100
-	1    0    0    -1
-$EndComp
 Wire Wire Line
 	2500 3500 2500 3350
@@
 NoConn ~ 5450 3100
 Text GLabel 6350 2750 2    60   Input ~ 0
-Output
+ITF-D_amplified_filtered_signal
+Text GLabel 2500 3350 0    60   Input ~ 0
+ITF-B_5v
+Text GLabel 2500 4100 0    60   Input ~ 0
+ITF-A_gnd
 $EndSCHEMATC
