File: modules/done-high_voltage/MDL-hvc_v1/src/MDL-hvc_v1.sch (KiCad schematic (older format))
At the start: 34 parts, among them Q1 2N2222, Q2 2N2222, Q3 2N2907, U1 LM555N

Commit message: update modules
Connections:
- net VCC: no longer Q2.3 (C), R1.2, R4.1, U1.4 (R)
- net Output renamed -100V
- new net ITF-B_5v: R1.2, U1.4 (R)
- new net ITF-l_18V_alimentation: Q2.3 (C), R4.1
Changed lines of the file:
@@
 LIBS:valves
 LIBS:echopen
-LIBS:MDL_HVC_V1-cache
+LIBS:MDL-hvc_v1-cache
 EELAYER 25 0
 EELAYER END
@@
 Text Label 7400 7500 0    60   ~ 0
 Alimentation_Symétrique_+/-_5V;12V
-Text Label 3200 1350 0    60   ~ 0
-18V
-$Comp
-L VCC #PWR01
-U 1 1 57A21CBB
-P 3450 1450
-F 0 "#PWR01" H 3450 1300 50  0001 C CNN
-F 1 "VCC" H 3450 1600 50  0000 C CNN
-F 2 "" H 3450 1450 50  0000 C CNN
-F 3 "" H 3450 1450 50  0000 C CNN
-	1    3450 1450
-	1    0    0    -1
-$EndComp
 Wire Wire Line
 	1450 2350 2100 2350
@@
 Connection ~ 5250 2250
 Wire Wire Line
-	4350 2150 4350 2900
+	4350 2150 4350 3000
 Wire Wire Line
 	5250 1850 5850 1850
@@
 	1    0    0    -1
 $EndComp
-Text Label 1200 2250 0    60   ~ 0
-5V
-$Comp
-L VCC #PWR02
-U 1 1 57A231C1
-P 1450 2350
-F 0 "#PWR02" H 1450 2200 50  0001 C CNN
-F 1 "VCC" H 1450 2500 50  0000 C CNN
-F 2 "" H 1450 2350 50  0000 C CNN
-F 3 "" H 1450 2350 50  0000 C CNN
-	1    1450 2350
-	1    0    0    -1
-$EndComp
 Wire Wire Line
 	1650 2350 1650 1550
@@
 	6300 2250 6300 2150
 $Comp
-L GND #PWR03
-U 1 1 57A26714
-P 4350 2900
-F 0 "#PWR03" H 4350 2650 50  0001 C CNN
-F 1 "GND" H 4350 2750 50  0000 C CNN
-F 2 "" H 4350 2900 50  0000 C CNN
-F 3 "" H 4350 2900 50  0000 C CNN
-	1    4350 2900
-	1    0    0    -1
-$EndComp
-$Comp
 L CP C4
 U 1 1 57A26CAB
@@
 	10900 2900 10750 2900
 Connection ~ 4350 2900
-Text GLabel 10900 3100 3    60   Input ~ 0
-Output
+Text GLabel 10900 3100 0    60   Input ~ 0
+-100V
 Wire Wire Line
 	10900 2900 10900 3100
@@
 	1    0    0    1
 $EndComp
+Text GLabel 1450 2350 0    60   Input ~ 0
+ITF-B_5v
+Text GLabel 3450 1450 0    60   Input ~ 0
+ITF-l_18V_alimentation
+Text GLabel 4350 3000 0    60   Input ~ 0
+ITF-A_gnd
 $EndSCHEMATC
