File: modules/done-high_voltage/MDL-hvc_v2/src/MDL-hvc_v2.sch (KiCad schematic (older format))
At the start: 2 parts, among them U1 R05-100B

Commit message: update modules
Connections:
- net +5V renamed ITF-B_5v
- net GND renamed ITF-A_grd
- net Vout renamed -100V
Changed lines of the file:
@@
 LIBS:valves
 LIBS:echopen
-LIBS:MDL_HVC_V2-cache
+LIBS:MDL-hvc_v2-cache
 EELAYER 25 0
 EELAYER END
@@
 Connection ~ 4450 3600
 Connection ~ 4450 2650
-$Comp
-L GND #PWR01
-U 1 1 57A307B6
-P 4350 3600
-F 0 "#PWR01" H 4350 3350 50  0001 C CNN
-F 1 "GND" H 4350 3450 50  0000 C CNN
-F 2 "" H 4350 3600 50  0000 C CNN
-F 3 "" H 4350 3600 50  0000 C CNN
-	1    4350 3600
-	1    0    0    -1
-$EndComp
 Wire Wire Line
 	5450 2650 5550 2650
 Connection ~ 5450 2650
-$Comp
-L +5V #PWR02
-U 1 1 57A3087B
-P 5550 2650
-F 0 "#PWR02" H 5550 2500 50  0001 C CNN
-F 1 "+5V" H 5550 2790 50  0000 C CNN
-F 2 "" H 5550 2650 50  0000 C CNN
-F 3 "" H 5550 2650 50  0000 C CNN
-	1    5550 2650
-	1    0    0    -1
-$EndComp
 $Comp
 L POT RV1
@@
 Connection ~ 5800 3350
 Text GLabel 5900 3350 2    60   Input ~ 0
-Vout
+-100V
+Text GLabel 4350 3600 0    60   Input ~ 0
+ITF-A_grd
+Text GLabel 5550 2650 2    60   Input ~ 0
+ITF-B_5v
 $EndSCHEMATC
