File: modules/done_envelope_detector/MDL-envelope_detector_v1/src/MDL-envelope_detector_v1.sch (KiCad schematic (older format))
At the start: 3 parts

Commit message: update modules
Connections:
- net GND renamed ITF-A_gnd
- net Input renamed ITF-D_amplified_filtered_signal
- net Output renamed ITF-E_signal_envelope
Changed lines of the file:
@@
 LIBS:contrib
 LIBS:valves
+LIBS:MDL-envelope_detector_v1-cache
 EELAYER 25 0
 EELAYER END
@@
 Wire Wire Line
 	3350 2500 3600 2500
-$Comp
-L GND #PWR1
-U 1 1 57A4D5CE
-P 3350 2500
-F 0 "#PWR1" H 3350 2250 50  0001 C CNN
-F 1 "GND" H 3350 2350 50  0000 C CNN
-F 2 "" H 3350 2500 50  0000 C CNN
-F 3 "" H 3350 2500 50  0000 C CNN
-	1    3350 2500
-	1    0    0    -1
-$EndComp
 Text GLabel 2950 2200 0    60   Input ~ 0
-Input
-Text GLabel 3600 2200 1    60   Input ~ 0
-Output
+ITF-D_amplified_filtered_signal
+Text GLabel 3600 2200 2    60   Input ~ 0
+ITF-E_signal_envelope
+Text GLabel 3350 2500 0    60   Input ~ 0
+ITF-A_gnd
 $EndSCHEMATC
