File: electronic/daughter_boards/DB-envelope_detector/DB-envelope_detector_v1/src/DB-envelope_detector_v1.kicad_pcb (KiCad board)
At the start: 2 copper layers, 19 x 52.1 mm, 4 parts, among them P1 CONN_01X19

Commit message: update src of DBs
Parts:
- C1: footprint Capacitors_ThroughHole:C_Disc_D3_P2.5 -> Echopen:C_TH_common
- D1: footprint Diodes_ThroughHole:Diode_DO-35_SOD27_Horizontal_RM10 -> Echopen:D_TH_common
- R1: footprint Resistors_ThroughHole:Resistor_Horizontal_RM10mm -> Echopen:Resistor_TH_common
- moved C1 2.54 mm to (144.8, 110.5)
Connections:
- P1 pad 10: (no net) -> Net-(P1-Pad10)
- P1 pad 11: (no net) -> Net-(P1-Pad11)
- P1 pad 12: (no net) -> Net-(P1-Pad12)
- P1 pad 13: (no net) -> Net-(P1-Pad13)
- P1 pad 14: (no net) -> Net-(P1-Pad14)
- P1 pad 15: (no net) -> Net-(P1-Pad15)
- P1 pad 16: (no net) -> Net-(P1-Pad16)
- P1 pad 17: (no net) -> Net-(P1-Pad17)
- P1 pad 18: (no net) -> Net-(P1-Pad18)
- P1 pad 19: (no net) -> Net-(P1-Pad19)
- P1 pad 2: (no net) -> Net-(P1-Pad2)
- P1 pad 3: (no net) -> Net-(P1-Pad3)
- P1 pad 6: (no net) -> Net-(P1-Pad6)
- P1 pad 7: (no net) -> Net-(P1-Pad7)
- P1 pad 8: (no net) -> Net-(P1-Pad8)
- P1 pad 9: (no net) -> Net-(P1-Pad9)
Routing:
- net Net-(C1-Pad1): track 27.0 -> 24.4 mm
Other:
- board text added: "DB-envelope_detector_v1"
- board text removed: "DB_Envelope_Detector_V1"
