File: electronic/daughter_boards/DB-filter/DB-filter_v1/src/DB-filter_v1.kicad_pcb (KiCad board)
At the start: 2 copper layers, 14 x 52.1 mm, 4 parts, among them P1 CONN_01X19

Commit message: update src of DBs
Parts:
- L1: footprint Inductors:INDUCTOR_V -> Echopen:INDUCTOR_TH_common
Other:
- board text added: "DB-filter_v1"
- board text removed: "DB_Filter_V1"
Changed lines of the file:
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@@
     (visible_elements 7FFFFFFF)
     (pcbplotparams
-      (layerselection 0x010f0_80000001)
+      (layerselection 0x010fc_80000001)
       (usegerberextensions true)
       (excludeedgelayer true)
@@
     (add_net "Net-(L1-Pad1)")
   )
+  (module Echopen:INDUCTOR_TH_common (layer F.Cu)
+    (at 92.71 86.36 180)
+    (descr "Inductor (vertical)")
+    (tags INDUCTOR)
+    (attr smd)
+    (fp_text reference L1 (at 0 1.905 180) (layer F.SilkS)
+      (effects (font (size 1 1) (thickness 0.15)))
+    )
+    (fp_text value 10u (at 0.09906 -1.99898 180) (layer F.Fab)
+      (effects (font (size 1 1) (thickness 0.15)))
+    )
+    (fp_circle (center 0 0) (end 3.81 0) (layer F.SilkS) (width 0.15))
+    (pad 1 thru_hole rect (at -2.54 0 180) (size 1.905 1.905) (drill 0.8128) (layers *.Cu *.Mask F.SilkS)
+      (net 3 "Net-(L1-Pad1)"))
+    (pad 2 thru_hole circle (at 2.54 0 180) (size 1.905 1.905) (drill 0.8128) (layers *.Cu *.Mask F.SilkS)
+      (net 1 "Net-(C1-Pad1)"))
+    (model Inductors.3dshapes/INDUCTOR_V.wrl
+      (at (xyz 0 0 0))
+      (scale (xyz 2 2 2))
+      (rotate (xyz 0 0 0))
+    )
+  )
   (module Echopen:C_TH_common (layer F.Cu)
     (at 90.17 78.74)
     (descr "Capacitor 6mm Disc, Pitch 5mm")
     (tags Capacitor)
+    (attr smd)
     (fp_text reference C1 (at 2.54 -1.27) (layer F.SilkS)
       (effects (font (size 1 1) (thickness 0.15)))
@@
     )
   )
-  (module Inductors:INDUCTOR_V (layer F.Cu)
-    (at 92.71 86.36 180)
-    (descr "Inductor (vertical)")
-    (tags INDUCTOR)
-    (fp_text reference L1 (at 0 1.99898 180) (layer F.SilkS)
-      (effects (font (size 1 1) (thickness 0.15)))
-    )
-    (fp_text value 10u (at 0.09906 -1.99898 180) (layer F.Fab)
-      (effects (font (size 1 1) (thickness 0.15)))
-    )
-    (fp_circle (center 0 0) (end 3.81 0) (layer F.SilkS) (width 0.15))
-    (pad 1 thru_hole rect (at -2.54 0 180) (size 1.905 1.905) (drill 0.8128) (layers *.Cu *.Mask F.SilkS)
-      (net 3 "Net-(L1-Pad1)"))
-    (pad 2 thru_hole circle (at 2.54 0 180) (size 1.905 1.905) (drill 0.8128) (layers *.Cu *.Mask F.SilkS)
-      (net 1 "Net-(C1-Pad1)"))
-    (model Inductors.3dshapes/INDUCTOR_V.wrl
-      (at (xyz 0 0 0))
-      (scale (xyz 2 2 2))
-      (rotate (xyz 0 0 0))
-    )
-  )
   (module Echopen:Header_pin_angled_1x19 (layer F.Cu)
     (at 86.36 86.36)
     (descr "Through hole socket strip")
     (tags "socket strip")
-    (fp_text reference P1 (at 2.54 -22.86) (layer F.SilkS)
+    (attr smd)
+    (fp_text reference P1 (at 3.81 -23.495) (layer F.SilkS)
       (effects (font (size 1 1) (thickness 0.15)))
     )
@@
     (descr "Resistor, Axial,  RM 10mm, 1/3W")
     (tags "Resistor Axial RM 10mm 1/3W")
+    (attr smd)
     (fp_text reference R1 (at 5.08 0 90) (layer F.SilkS)
       (effects (font (size 1 1) (thickness 0.15)))
     )
-    (fp_text value 330 (at 5.08 0 90) (layer F.Fab)
+    (fp_text value 330 (at 5.08 1.905 90) (layer F.Fab)
       (effects (font (size 1 1) (thickness 0.15)))
     )
@@
     )
   )
-  (gr_text DB_Filter_V1 (at 91.44 97.79 270) (layer B.SilkS)
+  (gr_text DB-filter_v1 (at 91.44 97.79 270) (layer B.SilkS)
     (effects (font (size 1.5 1.5) (thickness 0.3)) (justify mirror))
   )
