File: electronic/daughter_boards/DB-filter/DB-filter_v1/src/DB-filter_v1.sch (KiCad schematic (older format))
At the start: 4 parts, among them P1 CONN_01X19

Commit message: update src of DBs
Parts:
- C1: Caracteristic (none) -> 25V 10%; Manufacturer (none) -> AVX; Ref Manufacturer (none) -> SR151C102KAA
- L1: footprint Inductors:INDUCTOR_V -> Echopen:INDUCTOR_TH_common; Caracteristic (none) -> 10% 550mA; Manufacturer (none) -> Bourns; Ref Manufacturer (none) -> RLB0608-100KL
- P1: Caracteristic (none) -> angled pin header 1*19; Manufacturer (none) -> Molex; Ref Manufacturer (none) -> 22-28-8192
- R1: Caracteristic (none) -> 1/4W 5%; Manufacturer (none) -> KOA speer; Ref Manufacturer (none) -> MF1/4LCT52R331J
Changed lines of the file:
@@
 LIBS:valves
 LIBS:echopen
-LIBS:DB_Filter_V1-cache
+LIBS:DB-filter_v1-cache
 EELAYER 25 0
 EELAYER END
@@
 F 2 "Echopen:C_TH_common" H 4638 3000 50  0001 C CNN
 F 3 "" H 4600 3150 50  0000 C CNN
+F 4 "25V 10%" H 4600 3150 60  0001 C CNN "Caracteristic"
+F 5 "AVX" H 4600 3150 60  0001 C CNN "Manufacturer"
+F 6 "SR151C102KAA" H 4600 3150 60  0001 C CNN "Ref Manufacturer"
 	1    4600 3150
 	0    1    1    0
@@
 F 0 "L1" V 5000 3150 50  0000 C CNN
 F 1 "10u" V 5150 3150 50  0000 C CNN
-F 2 "Inductors:INDUCTOR_V" H 5050 3150 50  0001 C CNN
+F 2 "Echopen:INDUCTOR_TH_common" H 5050 3150 50  0001 C CNN
 F 3 "" H 5050 3150 50  0000 C CNN
+F 4 "10% 550mA" V 5050 3150 60  0001 C CNN "Caracteristic"
+F 5 "Bourns" V 5050 3150 60  0001 C CNN "Manufacturer"
+F 6 "RLB0608-100KL" V 5050 3150 60  0001 C CNN "Ref Manufacturer"
 	1    5050 3150
 	0    1    -1   0
@@
 F 2 "Echopen:Resistor_TH_common" V 5280 3300 50  0001 C CNN
 F 3 "" H 5350 3300 50  0000 C CNN
+F 4 "1/4W 5%" V 5350 3300 60  0001 C CNN "Caracteristic"
+F 5 "KOA speer" V 5350 3300 60  0001 C CNN "Manufacturer"
+F 6 "MF1/4LCT52R331J" V 5350 3300 60  0001 C CNN "Ref Manufacturer"
 	1    5350 3300
 	1    0    0    -1
@@
 F 2 "Echopen:Header_pin_angled_1x19" H 4100 3400 50  0001 C CNN
 F 3 "" H 4100 3400 50  0000 C CNN
+F 4 "angled pin header 1*19" H 4100 3400 60  0001 C CNN "Caracteristic"
+F 5 "Molex" H 4100 3400 60  0001 C CNN "Manufacturer"
+F 6 "22-28-8192" H 4100 3400 60  0001 C CNN "Ref Manufacturer"
 	1    4100 3400
 	-1   0    0    1
