File: electronic/daughter_boards/DB-high_voltage/DB-high_voltage_v1/src/DB-high_voltage_v1.kicad_pcb (KiCad board)
At the start: 2 copper layers, 53.3 x 52.1 mm, 37 parts, among them P1 CONN_01X19, P2 CONN_01X02, P3 SMA, Q1 Q2N2222, Q2 Q2N2222, Q3 Q2N2907, U1 LM555N

Commit message: update src of DBs
Parts:
- C1, C10, C11, C12, C13, C14, C2, C3, C4, C5, C6, C7, C8, C9: footprint Capacitors_ThroughHole:C_Radial_D5_L6_P2.5 -> Echopen:CP_small_TH_echopen
- D1, D12: value 1N4001 -> 1N4148
- D10, D11, D2, D3, D4, D5, D6, D7, D8, D9: value 1N5062 -> 1N4148
- P2: footprint Socket_Strips:Socket_Strip_Straight_1x02 -> Echopen:Socket_1x02
- Q1, Q2: value Q2N2222 -> 2N2222
- Q3: value Q2N2907 -> 2N2907
- U1: footprint Housings_DIP:DIP-8_W7.62mm -> Echopen:DIP-8(LM555)
Connections:
- P1 pad 10: (no net) -> Net-(P1-Pad10)
- P1 pad 11: (no net) -> Net-(P1-Pad11)
- P1 pad 13: (no net) -> Net-(P1-Pad13)
- P1 pad 14: (no net) -> Net-(P1-Pad14)
- P1 pad 15: (no net) -> Net-(P1-Pad15)
- P1 pad 16: (no net) -> Net-(P1-Pad16)
- P1 pad 17: (no net) -> Net-(P1-Pad17)
- P1 pad 18: (no net) -> Net-(P1-Pad18)
- P1 pad 19: (no net) -> Net-(P1-Pad19)
- P1 pad 3: (no net) -> Net-(P1-Pad3)
- P1 pad 4: (no net) -> Net-(P1-Pad4)
- P1 pad 5: (no net) -> Net-(P1-Pad5)
- P1 pad 6: (no net) -> Net-(P1-Pad6)
- P1 pad 7: (no net) -> Net-(P1-Pad7)
- P1 pad 8: (no net) -> Net-(P1-Pad8)
- P1 pad 9: (no net) -> Net-(P1-Pad9)
Other:
- board text added: "DB-high_voltage_v1"
- board text removed: "DB_HV_V1"
