File: electronic/daughter_boards/DB-motor_control/DB-motor_control_v2/src/DB-motor_control_v2.kicad_pcb (KiCad board)
At the start: 2 copper layers, 55.9 x 52.1 mm, 11 parts, among them P1 CONN_01X19, P2 CONN_01X15, P3 CONN_01X15, P4 CONN_01X08, P5 CONN_01X08, P6 CONN_01X04, Q1 2N2222

Commit message: update src of DBs
Parts:
- P2, P3: footprint Socket_Strips:Socket_Strip_Straight_1x15 -> Echopen:Pin_Header_Straight_1x15
- P4, P5: footprint Socket_Strips:Socket_Strip_Straight_1x08 -> Echopen:Pin_Header_Straight_1x08
- P6: footprint Socket_Strips:Socket_Strip_Straight_1x04 -> Echopen:Pin_Header_Straight_1x04
- turned P2 to 0 degrees
- turned P3 to 0 degrees
- turned P4 to 0 degrees
- turned P5 to 0 degrees
- turned P6 to 0 degrees
Connections:
- P1 pad 12: (no net) -> Net-(P1-Pad12)
- P1 pad 13: (no net) -> Net-(P1-Pad13)
- P1 pad 14: (no net) -> Net-(P1-Pad14)
- P1 pad 15: (no net) -> Net-(P1-Pad15)
- P1 pad 16: (no net) -> Net-(P1-Pad16)
- P1 pad 17: (no net) -> Net-(P1-Pad17)
- P1 pad 18: (no net) -> Net-(P1-Pad18)
- P1 pad 3: (no net) -> Net-(P1-Pad3)
- P1 pad 4: (no net) -> Net-(P1-Pad4)
- P1 pad 5: (no net) -> Net-(P1-Pad5)
- P1 pad 7: (no net) -> Net-(P1-Pad7)
- P1 pad 8: (no net) -> Net-(P1-Pad8)
- P2 pad 1: (no net) -> Net-(P2-Pad1)
- P2 pad 10: (no net) -> Net-(P2-Pad10)
- P2 pad 11: (no net) -> Net-(P2-Pad11)
- P2 pad 13: (no net) -> Net-(P2-Pad13)
- P2 pad 15: (no net) -> Net-(P2-Pad15)
- P2 pad 2: (no net) -> Net-(P2-Pad2)
- P2 pad 3: (no net) -> Net-(P2-Pad3)
- P2 pad 4: (no net) -> Net-(P2-Pad4)
- P2 pad 5: (no net) -> Net-(P2-Pad5)
- P2 pad 6: (no net) -> Net-(P2-Pad6)
- P2 pad 7: (no net) -> Net-(P2-Pad7)
- P2 pad 8: (no net) -> Net-(P2-Pad8)
- P2 pad 9: (no net) -> Net-(P2-Pad9)
- P3 pad 1: (no net) -> Net-(P3-Pad1)
- P3 pad 11: (no net) -> Net-(P3-Pad11)
- P3 pad 12: (no net) -> Net-(P3-Pad12)
- P3 pad 13: (no net) -> Net-(P3-Pad13)
- P3 pad 14: (no net) -> Net-(P3-Pad14)
- P3 pad 15: (no net) -> Net-(P3-Pad15)
