File: electronic/daughter_boards/DB-pulser/DB-pulser_v1/src/DB-pulser_v1.kicad_pcb (KiCad board)
At the start: 2 copper layers, 50.8 x 52.1 mm, 29 parts, among them P1 CONN_01X19, P2 CONN_01X02, P4 CONN_01X02, P5 SMA, P6 SMA, P7 CONN_01X02, P8 SMA, Q1 2N2907, Q2 2N2222, Q3 2N2222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

Commit message: update src of DBs
Parts:
- C1, C2, C4, C5: footprint Capacitors_ThroughHole:C_Disc_D3_P2.5 -> Echopen:C_small_TH_echopen
- C3: footprint Capacitors_ThroughHole:C_Radial_D10_L13_P5 -> Echopen:CP_TH_common
- D1: value BAT48 0.6V -> BAT48
- D2, D5: value BZD23-18 -> 1N4746
- D3: value D1N4148 -> 1N4148
- P2, P4, P7: footprint Socket_Strips:Socket_Strip_Angled_1x02 -> Echopen:Socket_1x02
- Q7, Q8: footprint TO_SOT_Packages_THT:TO-220_Neutral123_Vertical -> Echopen:TO-220_TH_common
Connections:
- P1 pad 10: (no net) -> Net-(P1-Pad10)
- P1 pad 11: (no net) -> Net-(P1-Pad11)
- P1 pad 12: (no net) -> Net-(P1-Pad12)
- P1 pad 13: (no net) -> Net-(P1-Pad13)
- P1 pad 14: (no net) -> Net-(P1-Pad14)
- P1 pad 15: (no net) -> Net-(P1-Pad15)
- P1 pad 16: (no net) -> Net-(P1-Pad16)
- P1 pad 17: (no net) -> Net-(P1-Pad17)
- P1 pad 18: (no net) -> Net-(P1-Pad18)
- P1 pad 19: (no net) -> Net-(P1-Pad19)
- P1 pad 2: (no net) -> Net-(P1-Pad2)
- P1 pad 3: (no net) -> Net-(P1-Pad3)
- P1 pad 4: (no net) -> Net-(P1-Pad4)
- P1 pad 5: (no net) -> Net-(P1-Pad5)
- P1 pad 7: (no net) -> Net-(P1-Pad7)
- P1 pad 8: (no net) -> Net-(P1-Pad8)
Other:
- board text added: "DB-pulser_v1"
- board text removed: "DB_Pulser_V1"
