File: electronic/daughter_boards/DB-pulser/DB-pulser_v1/src/DB-pulser_v1.sch (KiCad schematic (older format))
At the start: 29 parts, among them P1 CONN_01X19, P2 CONN_01X02, P4 CONN_01X02, P5 SMA, P6 SMA, P7 CONN_01X02, P8 SMA, Q1 2N2907, Q2 2N2222, Q3 2N2222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

Commit message: update src of DBs
Parts:
- C1: footprint Echopen:C_TH_common -> Echopen:C_small_TH_echopen; Caracteristic (none) -> 25V 10%; Manufacturer (none) -> Xicon; Ref Manufacturer (none) -> 140-50N5-101J-TB-RC
- C2, C4: footprint Echopen:C_TH_common -> Echopen:C_small_TH_echopen; Caracteristic (none) -> 25V 20%; Manufacturer (none) -> Xicon; Ref Manufacturer (none) -> 21RZ310-RC
- C3: Caracteristic (none) -> 150V 20%; Manufacturer (none) -> Lelon; Ref Manufacturer (none) -> REA330M2CBK-1320P
- C5: footprint Echopen:C_TH_common -> Echopen:C_small_TH_echopen; Caracteristic (none) -> 25V 10%; Manufacturer (none) -> Vishay; Ref Manufacturer (none) -> K221K15X7RF5TL2
- D1: value BAT48 0.6V -> BAT48; Caracteristic (none) -> NA; Manufacturer (none) -> STMicroelectronics; Ref Manufacturer (none) -> BAT48
- D2, D5: value BZD23-18 -> 1N4746; Caracteristic (none) -> Zener 18V; Manufacturer (none) -> Vishay; Ref Manufacturer (none) -> 1N4746A-TR
- D3: Caracteristic (none) -> NA; Manufacturer (none) -> Fairchild Semiconductor; Ref Manufacturer (none) -> 1N4148
- P1: Caracteristic (none) -> NA; Manufacturer (none) -> Molex; Ref Manufacturer (none) -> 22-28-8192
- P2, P4: footprint Socket_Strips:Socket_Strip_Angled_1x02 -> Echopen:Socket_1x02; Caracteristic (none) -> angled socket 1*02; Manufacturer (none) -> Molex; Ref Manufacturer (none) -> 22-15-2026
- P5, P6, P8: Caracteristic (none) -> NA; Manufacturer (none) -> Johnson / Cinch Connectivity Solutions; Ref Manufacturer (none) -> 142-0701-801
- P7: footprint Socket_Strips:Socket_Strip_Angled_1x02 -> Echopen:Socket_1x02; Caracteristic (none) -> angle socket 1*02; Manufacturer (none) -> Molex; Ref Manufacturer (none) -> 22-15-2026
- Q1, Q4, Q6: Caracteristic (none) -> NA; Manufacturer (none) -> Central Semiconductor; Ref Manufacturer (none) -> 2N2907A
- Q2, Q3, Q5: Caracteristic (none) -> NA; Manufacturer (none) -> Central Semiconductor; Ref Manufacturer (none) -> 2N2222
- Q7: footprint TO_SOT_Packages_THT:TO-220_Neutral123_Vertical -> Echopen:TO-220_TH_common; Caracteristic (none) -> NA; Manufacturer (none) -> Vishay; Ref Manufacturer (none) -> IRF9610PBF
- Q8: footprint TO_SOT_Packages_THT:TO-220_Neutral123_Vertical -> Echopen:TO-220_TH_common; Caracteristic (none) -> NA; Manufacturer (none) -> Vishay; Ref Manufacturer (none) -> IRF610PBF
- R1: Caracteristic (none) -> 1/4W 5%; Manufacturer (none) -> Yageo; Ref Manufacturer (none) -> MFR-25FRF52-1K
- R2: Caracteristic (none) -> 1/4W 5%; Manufacturer (none) -> Yageo; Ref Manufacturer (none) -> CFR-25JR-52-22R
- R3, R5: Caracteristic (none) -> 1/4W 5%; Manufacturer (none) -> Yageo; Ref Manufacturer (none) -> MFR-25FBF52-1M
- R6: Caracteristic (none) -> 1/4W 10%; Manufacturer (none) -> Vishay; Ref Manufacturer (none) -> CCF07100KJKE36
