File: electronic/daughter_boards/DB-pulser/DB-pulser_v2/src/DB-pulser_v2.kicad_pcb (KiCad board)
At the start: 2 copper layers, 45.7 x 52.1 mm, 9 parts, among them P1 CONN_01X19, P2 CONN_01X02, P3 CONN_01X08, P4 SMA, P5 CONN_01X02, P6 CONN_01X02, P7 SMA, P8 SMA

Commit message: update src of DBs
Parts:
- P1: footprint Echopen:Header_pin_angled_1x19 -> Echopen:Header_pin_1x19
- P2, P5, P6: footprint Socket_Strips:Socket_Strip_Angled_1x02 -> Echopen:Socket_1x02
- P3: footprint Socket_Strips:Socket_Strip_Angled_1x08 -> Echopen:Socket_Strip_Straight_1x08
Connections:
- P1 pad 10: (no net) -> Net-(P1-Pad10)
- P1 pad 11: (no net) -> Net-(P1-Pad11)
- P1 pad 12: (no net) -> Net-(P1-Pad12)
- P1 pad 13: (no net) -> Net-(P1-Pad13)
- P1 pad 14: (no net) -> Net-(P1-Pad14)
- P1 pad 15: (no net) -> Net-(P1-Pad15)
- P1 pad 16: (no net) -> Net-(P1-Pad16)
- P1 pad 17: (no net) -> Net-(P1-Pad17)
- P1 pad 18: (no net) -> Net-(P1-Pad18)
- P1 pad 19: (no net) -> Net-(P1-Pad19)
- P1 pad 3: (no net) -> Net-(P1-Pad3)
- P1 pad 4: (no net) -> Net-(P1-Pad4)
- P1 pad 5: (no net) -> Net-(P1-Pad5)
- P1 pad 7: (no net) -> Net-(P1-Pad7)
Other:
- board text added: "DB-pulser_v2"
- board text removed: "DB_Pulser_V2"
