File: electronic/daughter_boards/DB-supply/DB-supply_v1/src/DB-supply_v1.sch (KiCad schematic (older format))
At the start: 29 parts, among them P1 CONN_01X19, Q1 2N2222, Q2 2N2222, Q3 2N2907, U1 LM555N, U2 LM2940T-12.0/NOPB, U3 LM2940T-5.0/NOPB, U4 LM1117T-3.3/NOPB, U5 LM2990T-12.0/NOPB, U6 LM2990T-5.0/NOPB

Commit message: update src of DBs
Parts:
- C1: Caracteristic (none) -> 25V 10%; Manufacturer (none) -> Vishay; Ref Manufacturer (none) -> K103K15X7RF5UH5
- C10, C4, C5, C6, C7, C8, C9: Caracteristic (none) -> 25V 20%; Manufacturer (none) -> Nichicon; Ref Manufacturer (none) -> UVR1E470MDD6
- C2: Caracteristic (none) -> 25V 10%; Manufacturer (none) -> Vishay; Ref Manufacturer (none) -> 1C10Z5U473M050B
- C3: Caracteristic (none) -> 25V 20%; Manufacturer (none) -> Cornell Dubilier - CDE; Ref Manufacturer (none) -> 227CKS025MGM
- D1, D4: Caracteristic (none) -> NA; Manufacturer (none) -> Fairchild Semiconductor; Ref Manufacturer (none) -> 1N4148
- D2: Caracteristic (none) -> green LED; Manufacturer (none) -> parallax; Ref Manufacturer (none) -> 350-00001
- D3: value 1N4001 -> 1N4148; Caracteristic (none) -> NA; Manufacturer (none) -> Fairchild Semiconductor; Ref Manufacturer (none) -> 1N4148
- P1: footprint Socket_Strips:Socket_Strip_Straight_1x19 -> Echopen:Header_pin_angled_1x19; Caracteristic (none) -> angled pin 1*19; Manufacturer (none) -> Molex; Ref Manufacturer (none) -> 22-28-8192
- Q1, Q2: Caracteristic (none) -> NA; Manufacturer (none) -> Central Semiconductor; Ref Manufacturer (none) -> 2N2222
- Q3: Caracteristic (none) -> NA; Manufacturer (none) -> Central Semiconductor; Ref Manufacturer (none) -> 2N2907A
- R1: Caracteristic (none) -> 1/4W 10%; Manufacturer (none) -> KOA speer; Ref Manufacturer (none) -> MF1/4LCT52R222J
- R2: Caracteristic (none) -> 1/4W 5%; Manufacturer (none) -> KOA speer; Ref Manufacturer (none) -> MF1/4LCT52R123J
- R3: Caracteristic (none) -> 1/4W 10%; Manufacturer (none) -> KOA speer; Ref Manufacturer (none) -> MF1/4LCT52R332J
- R4: Caracteristic (none) -> 1/4W 10%; Manufacturer (none) -> KOA speer; Ref Manufacturer (none) -> MF1/4LCT52R182G
- R5: Caracteristic (none) -> 1/4W 10%; Manufacturer (none) -> KOA speer; Ref Manufacturer (none) -> MF1/4LCT52R271J
- U1: footprint Housings_DIP:DIP-8_W7.62mm -> Echopen:DIP-8(LM555); Caracteristic (none) -> timer; Manufacturer (none) -> TI; Ref Manufacturer (none) -> LM555CN/NOPB
- U2: Caracteristic (none) -> 12V 1A voltage regulator; Manufacturer (none) -> TI; Ref Manufacturer (none) -> LM2940CT-12/NOPB
- U3: Caracteristic (none) -> 5V 1A voltage regulator; Manufacturer (none) -> TI; Ref Manufacturer (none) -> LM2940CT-5.0/NOPB
- U4: Caracteristic (none) -> 3.3V 1A voltage regulator; Manufacturer (none) -> TI; Ref Manufacturer (none) -> LM1117T-3.3/NOPB
- U5: Caracteristic (none) -> -12V 1A voltage regulator; Manufacturer (none) -> TI; Ref Manufacturer (none) -> LM2990T-12/NOPB
- U6: Caracteristic (none) -> -5V 1A voltage regulator; Manufacturer (none) -> TI; Ref Manufacturer (none) -> LM2990T-5.0/NOPB
Changed lines of the file:
@@
 LIBS:valves
 LIBS:echopen
-LIBS:DB_Supply_V1-cache
 EELAYER 25 0
 EELAYER END
@@
 F 0 "U1" H 3550 4250 50  0000 L CNN
 F 1 "LM555N" H 3550 3550 50  0000 L CNN
-F 2 "Housings_DIP:DIP-8_W7.62mm" H 3950 3900 50  0001 C CNN
+F 2 "Echopen:DIP-8(LM555)" H 3950 3900 50  0001 C CNN
 F 3 "" H 3950 3900 50  0000 C CNN
+F 4 "timer" H 3950 3900 60  0001 C CNN "Caracteristic"
+F 5 "TI" H 3950 3900 60  0001 C CNN "Manufacturer"
+F 6 "LM555CN/NOPB" H 3950 3900 60  0001 C CNN "Ref Manufacturer"
 	1    3950 3900
 	1    0    0    -1
@@
 F 2 "Echopen:C_TH_common" H 3538 4350 50  0001 C CNN
 F 3 "" H 3500 4500 50  0000 C CNN
+F 4 "25V 10%" H 3500 4500 60  0001 C CNN "Caracteristic"
+F 5 "Vishay" H 3500 4500 60  0001 C CNN "Manufacturer"
+F 6 "K103K15X7RF5UH5" H 3500 4500 60  0001 C CNN "Ref Manufacturer"
 	1    3500 4500
 	0    1    1    0
@@
 F 2 "Echopen:Resistor_TH_common" V 4680 3950 50  0001 C CNN
 F 3 "" H 4750 3950 50  0000 C CNN
+F 4 "1/4W 5%" V 4750 3950 60  0001 C CNN "Caracteristic"
+F 5 "KOA speer" V 4750 3950 60  0001 C CNN "Manufacturer"
+F 6 "MF1/4LCT52R123J" V 4750 3950 60  0001 C CNN "Ref Manufacturer"
 	1    4750 3950
 	1    0    0    -1
@@
 F 2 "Echopen:Resistor_TH_common" V 4430 3300 50  0001 C CNN
 F 3 "" H 4500 3300 50  0000 C CNN
+F 4 "1/4W 10%" V 4500 3300 60  0001 C CNN "Caracteristic"
+F 5 "KOA speer" V 4500 3300 60  0001 C CNN "Manufacturer"
+F 6 "MF1/4LCT52R222J" V 4500 3300 60  0001 C CNN "Ref Manufacturer"
 	1    4500 3300
 	0    1    1    0
@@
 F 2 "Echopen:D_TH_common" H 4900 5350 50  0001 C CNN
 F 3 "" H 4900 5350 50  0000 C CNN
+F 4 "NA" H 4900 5350 60  0001 C CNN "Caracteristic"
+F 5 "Fairchild Semiconductor" H 4900 5350 60  0001 C CNN "Manufacturer"
+F 6 "1N4148" H 4900 5350 60  0001 C CNN "Ref Manufacturer"
 	1    4900 5350
 	-1   0    0    -1
@@
 F 2 "Echopen:CP_TH_common" H 5088 5500 50  0001 C CNN
 F 3 "" H 5050 5650 50  0000 C CNN
+F 4 "25V 20%" H 5050 5650 60  0001 C CNN "Caracteristic"
+F 5 "Cornell Dubilier - CDE" H 5050 5650 60  0001 C CNN "Manufacturer"
+F 6 "227CKS025MGM" H 5050 5650 60  0001 C CNN "Ref Manufacturer"
 	1    5050 5650
 	1    0    0    -1
@@
 F 2 "Echopen:CP_TH_common" H 5888 5500 50  0001 C CNN
 F 3 "" H 5850 5650 50  0000 C CNN
+F 4 "25V 20%" H 5850 5650 60  0001 C CNN "Caracteristic"
+F 5 "Nichicon" H 5850 5650 60  0001 C CNN "Manufacturer"
+F 6 "UVR1E470MDD6" H 5850 5650 60  0001 C CNN "Ref Manufacturer"
 	1    5850 5650
 	1    0    0    -1
@@
 F 2 "Echopen:CP_TH_common" H 6688 5500 50  0001 C CNN
 F 3 "" H 6650 5650 50  0000 C CNN
+F 4 "25V 20%" H 6650 5650 60  0001 C CNN "Caracteristic"
+F 5 "Nichicon" H 6650 5650 60  0001 C CNN "Manufacturer"
+F 6 "UVR1E470MDD6" H 6650 5650 60  0001 C CNN "Ref Manufacturer"
 	1    6650 5650
 	1    0    0    -1
@@
 F 2 "Echopen:Resistor_TH_common" V 6730 5350 50  0001 C CNN
 F 3 "" H 6800 5350 50  0000 C CNN
+F 4 "1/4W 10%" V 6800 5350 60  0001 C CNN "Caracteristic"
+F 5 "KOA speer" V 6800 5350 60  0001 C CNN "Manufacturer"
+F 6 "MF1/4LCT52R271J" V 6800 5350 60  0001 C CNN "Ref Manufacturer"
 	1    6800 5350
 	0    1    1    0
@@
 F 2 "Echopen:D_TH_common" H 6950 5550 50  0001 C CNN
 F 3 "" H 6950 5550 50  0000 C CNN
+F 4 "green LED" H 6950 5550 60  0001 C CNN "Caracteristic"
+F 5 "parallax" H 6950 5550 60  0001 C CNN "Manufacturer"
+F 6 "350-00001" H 6950 5550 60  0001 C CNN "Ref Manufacturer"
 	1    6950 5550
 	0    -1   -1   0
@@
 F 2 "Echopen:Resistor_TH_common" V 5630 3350 50  0001 C CNN
 F 3 "" H 5700 3350 50  0000 C CNN
+F 4 "1/4W 10%" V 5700 3350 60  0001 C CNN "Caracteristic"
+F 5 "KOA speer" V 5700 3350 60  0001 C CNN "Manufacturer"
+F 6 "MF1/4LCT52R182G" V 5700 3350 60  0001 C CNN "Ref Manufacturer"
 	1    5700 3350
 	1    0    0    -1
@@
 F 2 "Echopen:CP_TH_common" H 7388 3450 50  0001 C CNN
 F 3 "" H 7350 3600 50  0000 C CNN
+F 4 "25V 20%" H 7350 3600 60  0001 C CNN "Caracteristic"
+F 5 "Nichicon" H 7350 3600 60  0001 C CNN "Manufacturer"
+F 6 "UVR1E470MDD6" H 7350 3600 60  0001 C CNN "Ref Manufacturer"
 	1    7350 3600
 	0    -1   -1   0
@@
 P 7500 3750
 F 0 "D3" H 7500 3850 50  0000 C CNN
-F 1 "1N4001" H 7500 3650 50  0000 C CNN
+F 1 "1N4148" H 7500 3650 50  0000 C CNN
 F 2 "Echopen:D_TH_common" H 7500 3750 50  0001 C CNN
 F 3 "" H 7500 3750 50  0000 C CNN
+F 4 "NA" H 7500 3750 60  0001 C CNN "Caracteristic"
+F 5 "Fairchild Semiconductor" H 7500 3750 60  0001 C CNN "Manufacturer"
+F 6 "1N4148" H 7500 3750 60  0001 C CNN "Ref Manufacturer"
 	1    7500 3750
 	0    -1   -1   0
@@
 F 2 "Echopen:D_TH_common" H 7650 3600 50  0001 C CNN
 F 3 "" H 7650 3600 50  0000 C CNN
+F 4 "NA" H 7650 3600 60  0001 C CNN "Caracteristic"
+F 5 "Fairchild Semiconductor" H 7650 3600 60  0001 C CNN "Manufacturer"
+F 6 "1N4148" H 7650 3600 60  0001 C CNN "Ref Manufacturer"
 	1    7650 3600
 	1    0    0    -1
@@
 F 2 "Echopen:CP_TH_common" H 7838 3600 50  0001 C CNN
 F 3 "" H 7800 3750 50  0000 C CNN
+F 4 "25V 20%" H 7800 3750 60  0001 C CNN "Caracteristic"
+F 5 "Nichicon" H 7800 3750 60  0001 C CNN "Manufacturer"
+F 6 "UVR1E470MDD6" H 7800 3750 60  0001 C CNN "Ref Manufacturer"
 	1    7800 3750
 	1    0    0    1
@@
 F 2 "Echopen:CP_TH_common" H 8638 3600 50  0001 C CNN
 F 3 "" H 8600 3750 50  0000 C CNN
+F 4 "25V 20%" H 8600 3750 60  0001 C CNN "Caracteristic"
+F 5 "Nichicon" H 8600 3750 60  0001 C CNN "Manufacturer"
+F 6 "UVR1E470MDD6" H 8600 3750 60  0001 C CNN "Ref Manufacturer"
 	1    8600 3750
 	1    0    0    1
@@
 F 2 "Echopen:Resistor_TH_common" V 5180 3700 50  0001 C CNN
 F 3 "" H 5250 3700 50  0000 C CNN
+F 4 "1/4W 10%" V 5250 3700 60  0001 C CNN "Caracteristic"
+F 5 "KOA speer" V 5250 3700 60  0001 C CNN "Manufacturer"
+F 6 "MF1/4LCT52R332J" V 5250 3700 60  0001 C CNN "Ref Manufacturer"
 	1    5250 3700
 	0    1    1    0
@@
 F 2 "Echopen:C_TH_common" H 4788 4200 50  0001 C CNN
 F 3 "" H 4750 4350 50  0000 C CNN
+F 4 "25V 10%" H 4750 4350 60  0001 C CNN "Caracteristic"
+F 5 "Vishay" H 4750 4350 60  0001 C CNN "Manufacturer"
+F 6 "1C10Z5U473M050B" H 4750 4350 60  0001 C CNN "Ref Manufacturer"
 	1    4750 4350
 	-1   0    0    1
@@
 F 2 "Echopen:CP_TH_common" H 9438 3600 50  0001 C CNN
 F 3 "" H 9400 3750 50  0000 C CNN
+F 4 "25V 20%" H 9400 3750 60  0001 C CNN "Caracteristic"
+F 5 "Nichicon" H 9400 3750 60  0001 C CNN "Manufacturer"
+F 6 "UVR1E470MDD6" H 9400 3750 60  0001 C CNN "Ref Manufacturer"
 	1    9400 3750
 	1    0    0    1
@@
 F 0 "P1" H 2350 5850 50  0000 C CNN
 F 1 "CONN_01X19" V 2450 4850 50  0000 C CNN
-F 2 "Socket_Strips:Socket_Strip_Straight_1x19" H 2350 4850 50  0001 C CNN
+F 2 "Echopen:Header_pin_angled_1x19" H 2350 4850 50  0001 C CNN
 F 3 "" H 2350 4850 50  0000 C CNN
+F 4 "angled pin 1*19" H 2350 4850 60  0001 C CNN "Caracteristic"
+F 5 "Molex" H 2350 4850 60  0001 C CNN "Manufacturer"
+F 6 "22-28-8192" H 2350 4850 60  0001 C CNN "Ref Manufacturer"
 	1    2350 4850
 	-1   0    0    1
@@
 F 2 "Echopen:CP_TH_common" H 6738 4350 50  0001 C CNN
 F 3 "" H 6700 4500 50  0000 C CNN
+F 4 "25V 20%" H 6700 4500 60  0001 C CNN "Caracteristic"
+F 5 "Nichicon" H 6700 4500 60  0001 C CNN "Manufacturer"
+F 6 "UVR1E470MDD6" H 6700 4500 60  0001 C CNN "Ref Manufacturer"
 	1    6700 4500
 	1    0    0    -1
@@
 F 2 "Echopen:TO-220_TH_common" H 5450 5400 50  0001 C CNN
 F 3 "" H 5450 5400 50  0000 C CNN
+F 4 "12V 1A voltage regulator" H 5450 5400 60  0001 C CNN "Caracteristic"
+F 5 "TI" H 5450 5400 60  0001 C CNN "Manufacturer"
+F 6 "LM2940CT-12/NOPB" H 5450 5400 60  0001 C CNN "Ref Manufacturer"
 	1    5450 5400
 	1    0    0    -1
@@
 F 2 "Echopen:TO-220_TH_common" H 6250 5400 50  0001 C CNN
 F 3 "" H 6250 5400 50  0000 C CNN
+F 4 "5V 1A voltage regulator" H 6250 5400 60  0001 C CNN "Caracteristic"
+F 5 "TI" H 6250 5400 60  0001 C CNN "Manufacturer"
+F 6 "LM2940CT-5.0/NOPB" H 6250 5400 60  0001 C CNN "Ref Manufacturer"
 	1    6250 5400
 	1    0    0    -1
@@
 F 2 "Echopen:TO-220_TH_common" H 6300 4400 50  0001 C CNN
 F 3 "" H 6300 4400 50  0000 C CNN
+F 4 "3.3V 1A voltage regulator" H 6300 4400 60  0001 C CNN "Caracteristic"
+F 5 "TI" H 6300 4400 60  0001 C CNN "Manufacturer"
+F 6 "LM1117T-3.3/NOPB" H 6300 4400 60  0001 C CNN "Ref Manufacturer"
 	1    6300 4400
 	1    0    0    -1
@@
 F 2 "Echopen:TO-18_TH_common" H 5800 3625 50  0001 L CIN
 F 3 "" H 5600 3700 50  0000 L CNN
+F 4 "NA" H 5600 3700 60  0001 C CNN "Caracteristic"
+F 5 "Central Semiconductor" H 5600 3700 60  0001 C CNN "Manufacturer"
+F 6 "2N2222" H 5600 3700 60  0001 C CNN "Ref Manufacturer"
 	1    5600 3700
 	1    0    0    -1
@@
 F 2 "Echopen:TO-18_TH_common" H 6700 3325 50  0001 L CIN
 F 3 "" H 6500 3400 50  0000 L CNN
+F 4 "NA" H 6500 3400 60  0001 C CNN "Caracteristic"
+F 5 "Central Semiconductor" H 6500 3400 60  0001 C CNN "Manufacturer"
+F 6 "2N2222" H 6500 3400 60  0001 C CNN "Ref Manufacturer"
 	1    6500 3400
 	1    0    0    -1
@@
 F 2 "Echopen:TO-18_TH_common" H 6800 3650 50  0001 L CIN
 F 3 "" H 6500 3800 50  0000 L CNN
+F 4 "NA" H 6500 3800 60  0001 C CNN "Caracteristic"
+F 5 "Central Semiconductor" H 6500 3800 60  0001 C CNN "Manufacturer"
+F 6 "2N2907A" H 6500 3800 60  0001 C CNN "Ref Manufacturer"
 	1    6500 3800
 	1    0    0    1
@@
 F 2 "Echopen:TO-220_TH_common" H 8200 3650 50  0001 C CNN
 F 3 "" H 8200 3650 50  0000 C CNN
+F 4 "-12V 1A voltage regulator" H 8200 3650 60  0001 C CNN "Caracteristic"
+F 5 "TI" H 8200 3650 60  0001 C CNN "Manufacturer"
+F 6 "LM2990T-12/NOPB" H 8200 3650 60  0001 C CNN "Ref Manufacturer"
 	1    8200 3650
 	1    0    0    -1
@@
 F 2 "Echopen:TO-220_TH_common" H 9000 3650 50  0001 C CNN
 F 3 "" H 9000 3650 50  0000 C CNN
+F 4 "-5V 1A voltage regulator" H 9000 3650 60  0001 C CNN "Caracteristic"
+F 5 "TI" H 9000 3650 60  0001 C CNN "Manufacturer"
+F 6 "LM2990T-5.0/NOPB" H 9000 3650 60  0001 C CNN "Ref Manufacturer"
 	1    9000 3650
 	1    0    0    -1
