File: electronic/daughter_boards/DB-supply/DB-supply_v1/src/DB-supply_v1.kicad_pcb (KiCad board)
At the start: 2 copper layers, 54.6 x 52.1 mm, 29 parts, among them P1 CONN_01X19, Q1 2N2222, Q2 2N2222, Q3 2N2907, U1 LM555N, U2 LM2940T-12.0/NOPB, U3 LM2940T-5.0/NOPB, U4 LM1117T-3.3/NOPB, U5 LM2990T-12.0/NOPB, U6 LM2990T-5.0/NOPB

Commit message: adding motor_control_v3
Parts:
- D3: value 1N4001 -> 1N4148
- U1: footprint Housings_DIP:DIP-8_W7.62mm -> Echopen:DIP-8(LM555)
Connections:
- P1 pad 10: (no net) -> Net-(P1-Pad10)
- P1 pad 11: (no net) -> Net-(P1-Pad11)
- P1 pad 13: (no net) -> Net-(P1-Pad13)
- P1 pad 14: (no net) -> Net-(P1-Pad14)
- P1 pad 15: (no net) -> Net-(P1-Pad15)
- P1 pad 16: (no net) -> Net-(P1-Pad16)
- P1 pad 17: (no net) -> Net-(P1-Pad17)
- P1 pad 3: (no net) -> Net-(P1-Pad3)
- P1 pad 4: (no net) -> Net-(P1-Pad4)
- P1 pad 5: (no net) -> Net-(P1-Pad5)
- P1 pad 7: (no net) -> Net-(P1-Pad7)
- P1 pad 9: (no net) -> Net-(P1-Pad9)
Other:
- board text added: "DB-supply_v1"
- board text removed: "DB_Supply_V1"
