File: electronic/daughter_boards/DB-tr_switch_tgc/DB-tr_switch_tgc_v1/src/DB-tr_switch_tgc_v1.kicad_pcb (KiCad board)
At the start: 2 copper layers, 41.9 x 52.1 mm, 15 parts, among them P1 CONN_01X19, P2 CONN_01X02, P3 SMA, P6 CONN_01X02, P7 CONN_01X02, P8 SMA, P9 SMA, U1 MD0100

Commit message: update src of DBs
Parts:
- D2: value IN4148 -> 1N4148
- P2, P6, P7: footprint Socket_Strips:Socket_Strip_Angled_1x02 -> Echopen:Socket_1x02
- W1, W2: footprint Measurement_Points:Test_Point_Keystone_5000-5004_Miniature -> Echopen:Test_Point
Connections:
- P1 pad 10: (no net) -> Net-(P1-Pad10)
- P1 pad 11: (no net) -> Net-(P1-Pad11)
- P1 pad 12: (no net) -> Net-(P1-Pad12)
- P1 pad 13: (no net) -> Net-(P1-Pad13)
- P1 pad 14: (no net) -> Net-(P1-Pad14)
- P1 pad 15: (no net) -> Net-(P1-Pad15)
- P1 pad 16: (no net) -> Net-(P1-Pad16)
- P1 pad 17: (no net) -> Net-(P1-Pad17)
- P1 pad 19: (no net) -> Net-(P1-Pad19)
- P1 pad 4: (no net) -> Net-(P1-Pad4)
- P1 pad 5: (no net) -> Net-(P1-Pad5)
- P1 pad 6: (no net) -> Net-(P1-Pad6)
- P1 pad 7: (no net) -> Net-(P1-Pad7)
- P1 pad 8: (no net) -> Net-(P1-Pad8)
- P1 pad 9: (no net) -> Net-(P1-Pad9)
Other:
- board text added: "DB-tr_switch_tgc_v1"
- board text removed: "DB_TRS_TGC_V1"
