File: electronic/daughter_boards/DB-tr_switch_tgc/DB-tr_switch_tgc_v1/src/DB-tr_switch_tgc_v1.sch (KiCad schematic (older format))
At the start: 15 parts, among them P1 CONN_01X19, P2 CONN_01X02, P3 SMA, P6 CONN_01X02, P7 CONN_01X02, P8 SMA, P9 SMA, U1 MD0100

Commit message: update src of DBs
Parts:
- AOP1: Caracteristic (none) -> high speed OPA; Manufacturer (none) -> TI; Ref Manufacturer (none) -> OPA625IDBVT
- C1: Caracteristic (none) -> 25V 10%; Manufacturer (none) -> AVX; Ref Manufacturer (none) -> SR151C102KAA
- D1, D2: Caracteristic (none) -> high speed diode; Manufacturer (none) -> Fairchild Semiconductor; Ref Manufacturer (none) -> 1N4148
- P1: footprint Socket_Strips:Socket_Strip_Straight_1x19 -> Echopen:Header_pin_angled_1x19; Caracteristic (none) -> angled pin 1*19; Manufacturer (none) -> Molex; Ref Manufacturer (none) -> 22-28-8192
- P2, P6: footprint Socket_Strips:Socket_Strip_Angled_1x02 -> Echopen:Socket_1x02; Caracteristic (none) -> angled socket 1*02; Manufacturer (none) -> Molex; Ref Manufacturer (none) -> 22-15-2026
- P3, P8, P9: Caracteristic (none) -> NA; Manufacturer (none) -> Johnson / Cinch Connectivity Solutions; Ref Manufacturer (none) -> 142-0701-801
- P7: footprint Socket_Strips:Socket_Strip_Angled_1x02 -> Echopen:Socket_1x02
- R1: Caracteristic (none) -> 1/4W 5%; Manufacturer (none) -> Yageo; Ref Manufacturer (none) -> CFR-25JB-52-220R
- U1: Caracteristic (none) -> NA; Manufacturer (none) -> Microchip Technology; Ref Manufacturer (none) -> MD0100N8-G
- W1, W2: footprint Measurement_Points:Test_Point_Keystone_5000-5004_Miniature -> Echopen:Test_Point; Caracteristic (none) -> test point; Manufacturer (none) -> Keystone Electronics; Ref Manufacturer (none) -> 5000
Changed lines of the file:
@@
 LIBS:valves
 LIBS:echopen
-LIBS:DB_TRS_TGC_V1-cache
 EELAYER 25 0
 EELAYER END
@@
 F 2 "Echopen:SOT89-3_(MD0100)" H 4450 2900 60  0001 C CNN
 F 3 "" H 4450 2900 60  0000 C CNN
+F 4 "NA" H 4450 2900 60  0001 C CNN "Caracteristic"
+F 5 "Microchip Technology" H 4450 2900 60  0001 C CNN "Manufacturer"
+F 6 "MD0100N8-G" H 4450 2900 60  0001 C CNN "Ref Manufacturer"
 	1    4450 2900
 	1    0    0    -1
@@
 F 2 "Echopen:D_TH_common" H 5050 3000 50  0001 C CNN
 F 3 "" H 5050 3000 50  0000 C CNN
+F 4 "high speed diode" H 5050 3000 60  0001 C CNN "Caracteristic"
+F 5 "Fairchild Semiconductor" H 5050 3000 60  0001 C CNN "Manufacturer"
+F 6 "1N4148" H 5050 3000 60  0001 C CNN "Ref Manufacturer"
 	1    5050 3000
 	0    1    1    0
@@
 F 2 "Echopen:D_TH_common" H 5350 3000 50  0001 C CNN
 F 3 "" H 5350 3000 50  0000 C CNN
+F 4 "high speed diode" H 5350 3000 60  0001 C CNN "Caracteristic"
+F 5 "Fairchild Semiconductor" H 5350 3000 60  0001 C CNN "Manufacturer"
+F 6 "1N4148" H 5350 3000 60  0001 C CNN "Ref Manufacturer"
 	1    5350 3000
 	0    1    -1   0
@@
 F 0 "P1" H 3000 3700 50  0000 C CNN
 F 1 "CONN_01X19" V 3100 2700 50  0000 C CNN
-F 2 "Socket_Strips:Socket_Strip_Straight_1x19" H 3000 2700 50  0001 C CNN
+F 2 "Echopen:Header_pin_angled_1x19" H 3000 2700 50  0001 C CNN
 F 3 "" H 3000 2700 50  0000 C CNN
+F 4 "angled pin 1*19" H 3000 2700 60  0001 C CNN "Caracteristic"
+F 5 "Molex" H 3000 2700 60  0001 C CNN "Manufacturer"
+F 6 "22-28-8192" H 3000 2700 60  0001 C CNN "Ref Manufacturer"
 	1    3000 2700
 	-1   0    0    1
@@
 F 2 "Echopen:SMA" H 3950 1850 50  0001 C CNN
 F 3 "" H 3950 1850 50  0000 C CNN
+F 4 "NA" H 3950 1850 60  0001 C CNN "Caracteristic"
+F 5 "Johnson / Cinch Connectivity Solutions" H 3950 1850 60  0001 C CNN "Manufacturer"
+F 6 "142-0701-801" H 3950 1850 60  0001 C CNN "Ref Manufacturer"
 	1    3950 1850
 	1    0    0    -1
@@
 F 0 "P2" H 3550 2050 50  0000 C CNN
 F 1 "CONN_01X02" V 3650 1900 50  0000 C CNN
-F 2 "Socket_Strips:Socket_Strip_Angled_1x02" H 3550 1900 50  0001 C CNN
+F 2 "Echopen:Socket_1x02" H 3550 1900 50  0001 C CNN
 F 3 "" H 3550 1900 50  0000 C CNN
+F 4 "angled socket 1*02" H 3550 1900 60  0001 C CNN "Caracteristic"
+F 5 "Molex" H 3550 1900 60  0001 C CNN "Manufacturer"
+F 6 "22-15-2026" H 3550 1900 60  0001 C CNN "Ref Manufacturer"
 	1    3550 1900
 	-1   0    0    -1
@@
 F 2 "Echopen:C_TH_common" H 5688 2700 50  0001 C CNN
 F 3 "" H 5650 2850 50  0000 C CNN
+F 4 "25V 10%" H 5650 2850 60  0001 C CNN "Caracteristic"
+F 5 "AVX" H 5650 2850 60  0001 C CNN "Manufacturer"
+F 6 "SR151C102KAA" H 5650 2850 60  0001 C CNN "Ref Manufacturer"
 	1    5650 2850
 	0    1    1    0
@@
 F 2 "Echopen:Resistor_TH_common" V 5830 3250 50  0001 C CNN
 F 3 "" H 5900 3250 50  0000 C CNN
+F 4 "1/4W 5%" V 5900 3250 60  0001 C CNN "Caracteristic"
+F 5 "Yageo" V 5900 3250 60  0001 C CNN "Manufacturer"
+F 6 "CFR-25JB-52-220R" V 5900 3250 60  0001 C CNN "Ref Manufacturer"
 	1    5900 3250
 	1    0    0    -1
@@
 F 2 "Echopen:SOT-23-6_Handsoldering(OPA625)" H 6450 2550 60  0001 C CNN
 F 3 "" H 6450 2550 60  0000 C CNN
+F 4 "high speed OPA" H 6500 2550 60  0001 C CNN "Caracteristic"
+F 5 "TI" H 6500 2550 60  0001 C CNN "Manufacturer"
+F 6 "OPA625IDBVT" H 6500 2550 60  0001 C CNN "Ref Manufacturer"
 	1    6500 2550
 	1    0    0    -1
@@
 F 2 "Echopen:SMA" H 7950 2150 50  0001 C CNN
 F 3 "" H 7950 2150 50  0000 C CNN
+F 4 "NA" H 7950 2150 60  0001 C CNN "Caracteristic"
+F 5 "Johnson / Cinch Connectivity Solutions" H 7950 2150 60  0001 C CNN "Manufacturer"
+F 6 "142-0701-801" H 7950 2150 60  0001 C CNN "Ref Manufacturer"
 	1    7950 2150
 	1    0    0    -1
@@
 F 0 "P6" H 7550 2350 50  0000 C CNN
 F 1 "CONN_01X02" V 7650 2200 50  0000 C CNN
-F 2 "Socket_Strips:Socket_Strip_Angled_1x02" H 7550 2200 50  0001 C CNN
+F 2 "Echopen:Socket_1x02" H 7550 2200 50  0001 C CNN
 F 3 "" H 7550 2200 50  0000 C CNN
+F 4 "angled socket 1*02" H 7550 2200 60  0001 C CNN "Caracteristic"
+F 5 "Molex" H 7550 2200 60  0001 C CNN "Manufacturer"
+F 6 "22-15-2026" H 7550 2200 60  0001 C CNN "Ref Manufacturer"
 	1    7550 2200
 	-1   0    0    -1
@@
 F 2 "Echopen:SMA" H 7950 3100 50  0001 C CNN
 F 3 "" H 7950 3100 50  0000 C CNN
+F 4 "NA" H 7950 3100 60  0001 C CNN "Caracteristic"
+F 5 "Johnson / Cinch Connectivity Solutions" H 7950 3100 60  0001 C CNN "Manufacturer"
+F 6 "142-0701-801" H 7950 3100 60  0001 C CNN "Ref Manufacturer"
 	1    7950 3100
 	1    0    0    -1
@@
 F 0 "P7" H 7550 3300 50  0000 C CNN
 F 1 "CONN_01X02" V 7650 3150 50  0000 C CNN
-F 2 "Socket_Strips:Socket_Strip_Angled_1x02" H 7550 3150 50  0001 C CNN
+F 2 "Echopen:Socket_1x02" H 7550 3150 50  0001 C CNN
 F 3 "" H 7550 3150 50  0000 C CNN
 	1    7550 3150
@@
 F 0 "W1" H 5450 3120 50  0000 C CNN
 F 1 "TEST_1P" H 5450 3050 50  0000 C CNN
-F 2 "Measurement_Points:Test_Point_Keystone_5000-5004_Miniature" H 5650 2850 50  0001 C CNN
+F 2 "Echopen:Test_Point" H 5650 2850 50  0001 C CNN
 F 3 "" H 5650 2850 50  0000 C CNN
+F 4 "test point" H 5450 2850 60  0001 C CNN "Caracteristic"
+F 5 "Keystone Electronics" H 5450 2850 60  0001 C CNN "Manufacturer"
+F 6 "5000" H 5450 2850 60  0001 C CNN "Ref Manufacturer"
 	1    5450 2850
 	1    0    0    -1
@@
 F 0 "W2" H 7250 2820 50  0000 C CNN
 F 1 "TEST_1P" H 7250 2750 50  0000 C CNN
-F 2 "Measurement_Points:Test_Point_Keystone_5000-5004_Miniature" H 7450 2550 50  0001 C CNN
+F 2 "Echopen:Test_Point" H 7450 2550 50  0001 C CNN
 F 3 "" H 7450 2550 50  0000 C CNN
+F 4 "test point" H 7250 2550 60  0001 C CNN "Caracteristic"
+F 5 "Keystone Electronics" H 7250 2550 60  0001 C CNN "Manufacturer"
+F 6 "5000" H 7250 2550 60  0001 C CNN "Ref Manufacturer"
 	1    7250 2550
 	1    0    0    -1
