File: electronic/daughter_boards/DB-motor_control/DB-motor_control_v3/src/DB-motor_control_v3_old.kicad_pcb (KiCad board)
At the start: 2 copper layers, 64.8 x 52.1 mm, 17 parts, among them P1 CONN_01X19, P2 CONN_01X09, P3 CONN_01X08, P4 CONN_01X08, P5 CONN_01X04, P6 CONN_01X15, P7 CONN_01X15, Q1 2N2222, Q2 2N2222

Commit message: correct MDL pulser and update DB motor control
Parts:
- turned P2 to 270 degrees
Routing:
- net Net-(P2-Pad9): track 7.62 -> 0.00 mm
- net Net-(P2-Pad7): track 9.72 -> 14.8 mm
- net GND: track 0.00 -> 4.86 mm, vias 0 -> 1
- net Net-(P2-Pad3): track 15.0 -> 12.7 mm, vias 1 -> 0
Changed lines of the file:
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@@
   (general
     (links 40)
-    (no_connects 13)
-    (area 79.934999 83.744999 144.855001 135.965001)
+    (no_connects 15)
+    (area 78.151667 83.744999 147.273334 150.215001)
     (thickness 1.6)
     (drawings 4)
@@
   )
   (module Echopen:Socket_1x09 (layer F.Cu)
-    (at 91.44 114.3)
+    (at 91.44 114.3 270)
     (descr "Through hole socket strip")
     (tags "socket strip")
-    (fp_text reference P2 (at 0 -5.1) (layer F.SilkS)
-      (effects (font (size 1 1) (thickness 0.15)))
-    )
-    (fp_text value CONN_01X09 (at 0 -3.1) (layer F.Fab)
+    (fp_text reference P2 (at 0 -5.1 270) (layer F.SilkS)
+      (effects (font (size 1 1) (thickness 0.15)))
+    )
+    (fp_text value CONN_01X09 (at 0 -3.1 270) (layer F.Fab)
       (effects (font (size 1 1) (thickness 0.15)))
     )
@@
     (fp_line (start 0 -1.55) (end -1.55 -1.55) (layer F.SilkS) (width 0.15))
     (fp_line (start -1.55 -1.55) (end -1.55 1.55) (layer F.SilkS) (width 0.15))
-    (pad 1 thru_hole circle (at 0 0) (size 2.2 2.2) (drill 1.016) (layers *.Cu *.Mask)
+    (pad 1 thru_hole circle (at 0 0 270) (size 2.2 2.2) (drill 1.016) (layers *.Cu *.Mask)
       (net 20 "Net-(P2-Pad1)"))
-    (pad 2 thru_hole circle (at 2.54 0) (size 2.2 2.2) (drill 1.016) (layers *.Cu *.Mask)
-      (net 2 GND))
-    (pad 3 thru_hole circle (at 5.08 0) (size 2.2 2.2) (drill 1.016) (layers *.Cu *.Mask)
+    (pad 2 thru_hole circle (at 2.54 0 270) (size 2.2 2.2) (drill 1.016) (layers *.Cu *.Mask)
+      (net 2 GND))
+    (pad 3 thru_hole circle (at 5.08 0 270) (size 2.2 2.2) (drill 1.016) (layers *.Cu *.Mask)
       (net 7 "Net-(P2-Pad3)"))
-    (pad 4 thru_hole circle (at 7.62 0) (size 2.2 2.2) (drill 1.016) (layers *.Cu *.Mask)
+    (pad 4 thru_hole circle (at 7.62 0 270) (size 2.2 2.2) (drill 1.016) (layers *.Cu *.Mask)
       (net 8 "Net-(P2-Pad4)"))
-    (pad 5 thru_hole circle (at 10.16 0) (size 2.2 2.2) (drill 1.016) (layers *.Cu *.Mask)
+    (pad 5 thru_hole circle (at 10.16 0 270) (size 2.2 2.2) (drill 1.016) (layers *.Cu *.Mask)
       (net 9 "Net-(P2-Pad5)"))
-    (pad 6 thru_hole circle (at 12.7 0) (size 2.2 2.2) (drill 1.016) (layers *.Cu *.Mask)
+    (pad 6 thru_hole circle (at 12.7 0 270) (size 2.2 2.2) (drill 1.016) (layers *.Cu *.Mask)
       (net 10 "Net-(P2-Pad6)"))
-    (pad 7 thru_hole circle (at 15.24 0) (size 2.2 2.2) (drill 1.016) (layers *.Cu *.Mask)
+    (pad 7 thru_hole circle (at 15.24 0 270) (size 2.2 2.2) (drill 1.016) (layers *.Cu *.Mask)
       (net 11 "Net-(P2-Pad7)"))
-    (pad 8 thru_hole circle (at 17.78 0) (size 2.2 2.2) (drill 1.016) (layers *.Cu *.Mask)
+    (pad 8 thru_hole circle (at 17.78 0 270) (size 2.2 2.2) (drill 1.016) (layers *.Cu *.Mask)
       (net 12 "Net-(P2-Pad8)"))
-    (pad 9 thru_hole circle (at 20.32 0) (size 2.2 2.2) (drill 1.016) (layers *.Cu *.Mask)
+    (pad 9 thru_hole circle (at 20.32 0 270) (size 2.2 2.2) (drill 1.016) (layers *.Cu *.Mask)
       (net 21 "Net-(P2-Pad9)"))
     (model Socket_Strips.3dshapes/Socket_Strip_Straight_1x09.wrl
@@
   (segment (start 88.9 88.9) (end 88.9 95.21) (width 0.25) (layer F.Cu) (net 1))
   (segment (start 88.9 95.21) (end 88.94 95.25) (width 0.25) (layer F.Cu) (net 1))
+  (segment (start 91.44 116.84) (end 92.71 116.84) (width 0.25) (layer B.Cu) (net 2))
+  (segment (start 92.71 116.84) (end 95.25 114.3) (width 0.25) (layer B.Cu) (net 2))
+  (via (at 95.25 114.3) (size 0.6) (drill 0.4) (layers F.Cu B.Cu) (net 2))
   (segment (start 104.14 88.9) (end 115.57 100.33) (width 0.25) (layer F.Cu) (net 3))
   (segment (start 114.3 114.3) (end 111.76 114.3) (width 0.25) (layer B.Cu) (net 3))
@@
   (segment (start 82.55 107.95) (end 127 107.95) (width 0.25) (layer B.Cu) (net 4))
   (segment (start 127 110.49) (end 82.55 110.49) (width 0.25) (layer B.Cu) (net 5))
-  (segment (start 91.44 116.84) (end 92.71 116.84) (width 0.25) (layer B.Cu) (net 7))
-  (segment (start 92.71 116.84) (end 95.25 114.3) (width 0.25) (layer B.Cu) (net 7))
-  (via (at 95.25 114.3) (size 0.6) (drill 0.4) (layers F.Cu B.Cu) (net 7))
   (segment (start 95.25 114.3) (end 95.25 104.14) (width 0.25) (layer F.Cu) (net 7))
-  (segment (start 91.44 119.38) (end 93.98 119.38) (width 0.25) (layer B.Cu) (net 8))
+  (segment (start 91.44 119.38) (end 93.98 119.38) (width 0.25) (layer B.Cu) (net 7))
   (segment (start 93.98 119.38) (end 99.06 114.3) (width 0.25) (layer B.Cu) (net 8))
-  (segment (start 91.44 121.92) (end 93.98 121.92) (width 0.25) (layer B.Cu) (net 9))
+  (segment (start 91.44 121.92) (end 93.98 121.92) (width 0.25) (layer B.Cu) (net 8))
   (segment (start 93.98 121.92) (end 99.06 116.84) (width 0.25) (layer B.Cu) (net 9))
-  (segment (start 91.44 124.46) (end 93.98 124.46) (width 0.25) (layer B.Cu) (net 10))
+  (segment (start 91.44 124.46) (end 93.98 124.46) (width 0.25) (layer B.Cu) (net 9))
   (segment (start 93.98 124.46) (end 99.06 119.38) (width 0.25) (layer B.Cu) (net 10))
-  (segment (start 91.44 127) (end 93.98 127) (width 0.25) (layer B.Cu) (net 11))
+  (segment (start 91.44 127) (end 93.98 127) (width 0.25) (layer B.Cu) (net 10))
   (segment (start 93.98 127) (end 99.06 121.92) (width 0.25) (layer B.Cu) (net 11))
-  (segment (start 91.44 129.54) (end 99.06 129.54) (width 0.25) (layer B.Cu) (net 12))
+  (segment (start 91.44 129.54) (end 99.06 129.54) (width 0.25) (layer B.Cu) (net 11))
+  (segment (start 91.44 132.08) (end 99.06 132.08) (width 0.25) (layer B.Cu) (net 12))
   (segment (start 99.06 127) (end 99.06 124.46) (width 0.25) (layer B.Cu) (net 13))
   (segment (start 111.76 119.38) (end 118.11 119.38) (width 0.25) (layer B.Cu) (net 14))
@@
   (segment (start 109.22 102.87) (end 113.03 102.87) (width 0.25) (layer B.Cu) (net 19))
   (segment (start 107.95 104.14) (end 109.22 102.87) (width 0.25) (layer B.Cu) (net 19))
-  (segment (start 91.44 132.08) (end 99.06 132.08) (width 0.25) (layer B.Cu) (net 21))
   (segment (start 105.41 100.33) (end 110.49 100.33) (width 0.25) (layer B.Cu) (net 22))
   (segment (start 110.49 100.33) (end 111.76 101.6) (width 0.25) (layer B.Cu) (net 22))
