File: electronic/daughter_boards/DB-motor_control/DB-motor_control_v3/src/DB-motor_control_v3.kicad_pcb (KiCad board)
At the start: 2 copper layers, 64.8 x 52.1 mm, 17 parts, among them P1 CONN_01X19, P2 CONN_01X09, P3 CONN_01X08, P4 CONN_01X08, P5 CONN_01X04, P6 CONN_01X15, P7 CONN_01X15, Q1 2N2222, Q2 2N2222

Commit message: adding motor_control_v3 documentation
Parts:
- added C5: 47n, Echopen:C_small_TH_echopen, F.Cu at (86.4, 126.4)
- added C6: 10u, Echopen:CP_small_TH_echopen, F.Cu at (87.6, 130.8)
- P2: footprint Echopen:Socket_1x09 -> Socket_Strips:Socket_Strip_Straight_1x09_Pitch2.54mm
- moved R3 7.73 mm to (87.6, 111.8)
- moved P2 1.27 mm to (92.7, 111.8), turned to 0 degrees
Connections:
- P1 pad 11: (no net) -> Net-(P1-Pad11)
- P1 pad 19: Net-(P1-Pad19) -> Net-(C5-Pad1)
- P2 pad 1: Net-(P2-Pad1) -> Net-(P1-Pad11)
- P4 pad 7: Net-(C1-Pad1) -> Net-(C5-Pad1)
- Q2 pad 3: Net-(P2-Pad1) -> Net-(P1-Pad11)
- R3 pad 1: Net-(P2-Pad1) -> Net-(P1-Pad11)
- R3 pad 2: Net-(P1-Pad19) -> Net-(C5-Pad1)
Routing:
- net Net-(P2-Pad1): track 59.6 -> 0.00 mm
- net Net-(P1-Pad11): track 0.00 -> 56.7 mm
- net Net-(C5-Pad1): track 0.00 -> 44.6 mm
- net Net-(C1-Pad1): track 120.9 -> 83.3 mm, vias 1 -> 0
- net Net-(P1-Pad19): track 6.13 -> 0.00 mm
- net GND: track 0.00 -> 1.80 mm
- net Net-(P2-Pad9): track 7.62 -> 6.35 mm
- net Net-(P2-Pad8): track 7.62 -> 6.35 mm
- net Net-(P2-Pad7): track 9.72 -> 8.45 mm
- net Net-(P2-Pad6): track 9.72 -> 8.45 mm
- net Net-(P2-Pad5): track 9.72 -> 8.45 mm
- net Net-(P2-Pad4): track 9.72 -> 8.45 mm
- net Net-(P2-Pad3): track 15.0 -> 13.8 mm
