File: electronic/daughter_boards/DB-pulser/DB-pulser_v3/src/DB-pulser_v3.kicad_pcb (KiCad board)
At the start: 2 copper layers, 47 x 52.1 mm, 16 parts, among them P1 CONN_01X19, P2 SMA, P3 CONN_01X02, P4 SMA, P5 SMA, P6 CONN_01X02, P7 CONN_01X02, U1 MOSFET_driver, U2 TC6320

Commit message: update instalation doc
Parts:
- added R1: 47, Echopen:Resistor_TH_common, F.Cu at (127.1, 128.9)
- U1: value MOSFET_driver -> MCP14A0154
Connections:
- P1 pad 10: Net-(P1-Pad10) -> (no net)
- P1 pad 11: Net-(P1-Pad11) -> (no net)
- P1 pad 12: Net-(P1-Pad12) -> (no net)
- P1 pad 13: Net-(P1-Pad13) -> (no net)
- P1 pad 14: Net-(P1-Pad14) -> (no net)
- P1 pad 15: Net-(P1-Pad15) -> (no net)
- P1 pad 16: Net-(P1-Pad16) -> (no net)
- P1 pad 17: Net-(P1-Pad17) -> (no net)
- P1 pad 18: Net-(P1-Pad18) -> (no net)
- P1 pad 19: Net-(P1-Pad19) -> (no net)
- P1 pad 2: Net-(P1-Pad2) -> (no net)
- P1 pad 3: Net-(P1-Pad3) -> (no net)
- P1 pad 4: Net-(P1-Pad4) -> (no net)
- P1 pad 5: Net-(P1-Pad5) -> (no net)
- P1 pad 7: Net-(P1-Pad7) -> (no net)
- P1 pad 8: Net-(P1-Pad8) -> (no net)
- U1 pad 1: Net-(U1-Pad1) -> (no net)
- U1 pad 8: Net-(U1-Pad8) -> (no net)
Routing:
- net Net-(D1-Pad1): track 59.5 -> 63.2 mm
